File: Kicad/Nanocomp6809V5/Nanocomp6809V5.kicad_sch (KiCad schematic)
At the start: 77 parts, among them J1 TTL_USB_Serial_FT232R, J2 DB15_Female_HighDensity, J3 Conn_01x15_Male, SW1 R, SW10 0, SW11 3, SW12 2, SW13 D, SW14 C, SW15 B, SW16 A, SW17 1, SW18 4, SW19 7, SW2 F, SW20 G, SW21 CN, SW22 S, SW23 L, SW24 RST, SW25 AB, SW3 6, SW4 5, SW5 M, SW6 E, SW7 9, SW8 8, SW9 I, U1 MC6809, U10 74LS92, U11 MC6850, U12 74LS245, U13 74LS541BB, U14 74LS541BB, U15 74LS541BB, U16 74LS241BB, U17 74LS157BB, U18 74LS166BB, U19 74LS04, U2 ATF22LV10, U20 REN7134-Memory_RAM, U21 74LS163-74xx, U22 74LS10, U23 MC6845BB, U24 REN7134-Memory_RAM, U3 28C64B, U4 AS6C1008, U5 6821_BBPIN, U6 7_Segment_x_4_LED_Nanocomp_RH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, U7 ULN2803A, U8 74LS145, U9 7_Segment_x_4_LED_Nanocomp, Y1 4Mhz, Y2 MXO45HS-3C-3M6862, Y3 MXO45HS-3C-25M1750

Commit message: Additional files for VGA videos V01-V04
Additional Datasheets, Assembly Source, fonts for first 4 VGA controller videos V01-V04
Connections:
- net Y0 is gone; now on net GND: U2.23 (I/O0), U20.5 (~{OE}L)
- net GND: now also R12.1, U24.43 (~{OE}R); no longer U24.47 (~{CE}R)
- net Y2: now also U24.47 (~{CE}R); no longer U24.43 (~{OE}R)
- net F/~{B} renamed DotOut
Changed lines of the file:
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@@
   (junction (at 135.89 85.09) (diameter 0) (color 0 0 0 0)
   )
-  (junction (at 78.74 161.29) (diameter 0) (color 0 0 0 0)
-  )
   (junction (at 575.31 120.65) (diameter 0) (color 0 0 0 0)
   )
@@
   (junction (at 78.74 67.31) (diameter 0) (color 0 0 0 0)
   )
-  (junction (at 237.49 162.56) (diameter 0) (color 0 0 0 0)
-  )
   (junction (at 349.25 254) (diameter 0) (color 0 0 0 0)
   )
@@
   (junction (at 358.14 199.39) (diameter 0) (color 0 0 0 0)
   )
+  (junction (at 66.04 74.93) (diameter 0) (color 0 0 0 0)
+  )
   (junction (at 119.38 52.07) (diameter 0) (color 0 0 0 0)
   )
@@
   (junction (at 365.76 207.01) (diameter 0) (color 0 0 0 0)
   )
+  (junction (at 237.49 173.99) (diameter 0) (color 0 0 0 0)
+  )
   (junction (at 346.71 74.93) (diameter 0) (color 0 0 0 0)
   )
@@
   (junction (at 349.25 77.47) (diameter 0) (color 0 0 0 0)
   )
+  (junction (at 78.74 172.72) (diameter 0) (color 0 0 0 0)
+  )
   (junction (at 63.5 62.23) (diameter 0) (color 0 0 0 0)
   )
@@
     (stroke (width 0) (type default) (color 0 0 0 0))
   )
-  (wire (pts (xy 224.79 172.72) (xy 224.79 173.99))
-    (stroke (width 0) (type default) (color 0 0 0 0))
-  )
   (wire (pts (xy 171.45 160.02) (xy 171.45 40.64))
     (stroke (width 0) (type default) (color 0 0 0 1))
@@
     (stroke (width 0) (type default) (color 0 0 0 0))
   )
-  (wire (pts (xy 78.74 111.76) (xy 78.74 161.29))
+  (wire (pts (xy 78.74 111.76) (xy 78.74 172.72))
     (stroke (width 0) (type default) (color 0 0 0 1))
   )
@@
     (stroke (width 0) (type default) (color 0 0 0 0))
   )
+  (wire (pts (xy 78.74 172.72) (xy 78.74 209.55))
+    (stroke (width 0) (type default) (color 0 0 0 1))
+  )
   (wire (pts (xy 81.28 34.29) (xy 81.28 44.45))
     (stroke (width 0) (type default) (color 255 0 0 1))
@@
     (stroke (width 0) (type default) (color 0 0 0 0))
   )
+  (wire (pts (xy 219.71 162.56) (xy 254 162.56))
+    (stroke (width 0) (type default) (color 0 0 0 0))
+  )
   (wire (pts (xy 317.5 156.21) (xy 328.93 156.21))
     (stroke (width 0) (type default) (color 0 0 0 0))
@@
     (stroke (width 0) (type default) (color 0 0 0 0))
   )
+  (wire (pts (xy 66.04 73.66) (xy 66.04 74.93))
+    (stroke (width 0) (type default) (color 0 0 0 0))
+  )
   (wire (pts (xy 281.94 77.47) (xy 288.29 77.47))
     (stroke (width 0) (type default) (color 255 0 0 1))
@@
     (stroke (width 0) (type default) (color 0 0 0 1))
   )
+  (wire (pts (xy 127 161.29) (xy 135.89 161.29))
+    (stroke (width 0) (type default) (color 0 0 0 0))
+  )
   (wire (pts (xy 139.7 64.77) (xy 134.62 64.77))
     (stroke (width 0) (type default) (color 0 0 0 0))
@@
     (stroke (width 0) (type default) (color 0 0 0 0))
   )
-  (wire (pts (xy 237.49 162.56) (xy 237.49 384.81))
-    (stroke (width 0) (type default) (color 0 0 0 1))
-  )
   (wire (pts (xy 483.87 115.57) (xy 487.68 115.57))
     (stroke (width 0) (type default) (color 0 0 0 0))
@@
     (stroke (width 0) (type default) (color 0 0 0 0))
   )
-  (wire (pts (xy 219.71 162.56) (xy 237.49 162.56))
-    (stroke (width 0) (type default) (color 0 0 0 0))
-  )
   (wire (pts (xy 506.73 124.46) (xy 518.16 124.46))
     (stroke (width 0) (type default) (color 0 0 0 0))
@@
     (stroke (width 0) (type default) (color 0 0 0 0))
   )
-  (wire (pts (xy 127 153.67) (xy 127 172.72))
-    (stroke (width 0) (type default) (color 0 0 0 0))
-  )
   (bus (pts (xy 402.59 149.86) (xy 405.13 149.86))
     (stroke (width 0) (type default) (color 0 0 0 0))
@@
     (stroke (width 0) (type default) (color 0 0 0 0))
   )
-  (wire (pts (xy 135.89 161.29) (xy 78.74 161.29))
-    (stroke (width 0) (type default) (color 0 0 0 0))
-  )
   (wire (pts (xy 116.84 46.99) (xy 130.81 46.99))
     (stroke (width 0) (type default) (color 0 0 0 0))
@@
     (stroke (width 0) (type default) (color 0 0 0 0))
   )
-  (wire (pts (xy 388.62 172.72) (xy 233.68 172.72))
+  (wire (pts (xy 388.62 172.72) (xy 254 172.72))
     (stroke (width 0) (type default) (color 0 0 0 0))
   )
@@
     (stroke (width 0) (type default) (color 0 0 0 0))
   )
-  (wire (pts (xy 15.24 22.86) (xy 36.83 22.86))
+  (wire (pts (xy 66.04 74.93) (xy 78.74 74.93))
     (stroke (width 0) (type default) (color 0 0 0 0))
   )
-  (wire (pts (xy 485.14 69.85) (xy 487.68 69.85))
+  (wire (pts (xy 15.24 22.86) (xy 36.83 22.86))
     (stroke (width 0) (type default) (color 0 0 0 0))
   )
-  (wire (pts (xy 224.79 173.99) (xy 233.68 173.99))
+  (wire (pts (xy 485.14 69.85) (xy 487.68 69.85))
     (stroke (width 0) (type default) (color 0 0 0 0))
   )
@@
     (stroke (width 0) (type default) (color 0 0 0 0))
   )
-  (wire (pts (xy 63.5 74.93) (xy 78.74 74.93))
+  (wire (pts (xy 63.5 74.93) (xy 66.04 74.93))
     (stroke (width 0) (type default) (color 0 0 0 0))
   )
@@
     (stroke (width 0) (type default) (color 0 0 0 0))
   )
-  (wire (pts (xy 130.81 172.72) (xy 127 172.72))
+  (wire (pts (xy 78.74 172.72) (xy 130.81 172.72))
     (stroke (width 0) (type default) (color 0 0 0 0))
   )
@@
     (stroke (width 0) (type default) (color 0 0 0 0))
   )
-  (wire (pts (xy 78.74 161.29) (xy 78.74 209.55))
-    (stroke (width 0) (type default) (color 0 0 0 1))
-  )
   (wire (pts (xy 487.68 74.93) (xy 492.76 74.93))
     (stroke (width 0) (type default) (color 0 0 0 0))
@@
     (stroke (width 0) (type default) (color 0 0 0 0))
   )
-  (wire (pts (xy 233.68 173.99) (xy 233.68 172.72))
-    (stroke (width 0) (type default) (color 0 0 0 0))
-  )
   (bus (pts (xy 388.62 29.21) (xy 386.08 29.21))
     (stroke (width 0) (type default) (color 0 0 0 0))
@@
     (stroke (width 0) (type default) (color 0 0 0 0))
   )
+  (wire (pts (xy 127 153.67) (xy 127 161.29))
+    (stroke (width 0) (type default) (color 0 0 0 0))
+  )
   (bus (pts (xy 335.28 72.39) (xy 337.82 72.39))
     (stroke (width 0) (type default) (color 0 0 0 0))
@@
     (stroke (width 0) (type default) (color 0 0 0 0))
   )
+  (wire (pts (xy 224.79 172.72) (xy 224.79 173.99))
+    (stroke (width 0) (type default) (color 0 0 0 0))
+  )
   (wire (pts (xy 344.17 269.24) (xy 351.79 269.24))
     (stroke (width 0) (type default) (color 0 0 0 0))
@@
     (stroke (width 0) (type default) (color 255 0 0 1))
   )
+  (wire (pts (xy 224.79 173.99) (xy 237.49 173.99))
+    (stroke (width 0) (type default) (color 0 0 0 0))
+  )
   (bus (pts (xy 342.9 104.14) (xy 342.9 149.86))
     (stroke (width 0) (type default) (color 0 0 0 0))
@@
     (stroke (width 0) (type default) (color 0 0 0 0))
   )
+  (wire (pts (xy 237.49 173.99) (xy 237.49 384.81))
+    (stroke (width 0) (type default) (color 0 0 0 1))
+  )
   (bus (pts (xy 549.91 139.7) (xy 549.91 142.24))
     (stroke (width 0) (type default) (color 0 0 0 0))
@@
     (stroke (width 0) (type default) (color 0 0 0 0))
   )
-  (wire (pts (xy 237.49 156.21) (xy 237.49 162.56))
+  (wire (pts (xy 237.49 156.21) (xy 237.49 173.99))
     (stroke (width 0) (type default) (color 0 0 0 1))
   )
@@
     (stroke (width 0) (type default) (color 0 0 0 0))
   )
+  (wire (pts (xy 254 172.72) (xy 254 162.56))
+    (stroke (width 0) (type default) (color 0 0 0 0))
+  )
   (wire (pts (xy 281.94 44.45) (xy 281.94 24.13))
     (stroke (width 0) (type default) (color 0 0 0 0))
@@
     (effects (font (size 1.27 1.27)) (justify left bottom))
   )
-  (label "Y2" (at 236.22 172.72 180)
+  (label "Y2" (at 233.68 162.56 180)
     (effects (font (size 1.27 1.27)) (justify right bottom))
   )
@@
     (effects (font (size 1.27 1.27)) (justify left bottom))
   )
+  (label "DotOut" (at 86.36 116.84 0)
+    (effects (font (size 1.27 1.27)) (justify left bottom))
+  )
   (label "A7" (at 132.08 191.77 0)
     (effects (font (size 1.27 1.27)) (justify left bottom))
@@
     (effects (font (size 1.27 1.27)) (justify left bottom))
   )
+  (label "DotOut" (at 118.11 217.17 0)
+    (effects (font (size 1.27 1.27)) (justify left bottom))
+  )
   (label "Y7" (at 367.03 99.06 0)
     (effects (font (size 1.27 1.27)) (justify left bottom))
@@
     (effects (font (size 1.27 1.27)) (justify left bottom))
   )
+  (label "Y0" (at 135.89 161.29 180)
+    (effects (font (size 1.27 1.27)) (justify right bottom))
+  )
   (label "BA" (at 485.14 69.85 0)
     (effects (font (size 1.27 1.27)) (justify left bottom))
@@
     (effects (font (size 1.27 1.27)) (justify left bottom))
   )
+  (label "Y2" (at 257.81 172.72 180)
+    (effects (font (size 1.27 1.27)) (justify right bottom))
+  )
   (symbol (lib_id "Breadboarding:MC6845BB") (at 205.74 66.04 0) (unit 1)
